File: EEG_BLE.kicad_sch (KiCad schematic)
At the start: 151 parts, among them J1 USB_C_Receptacle_PowerOnly_6P, P1 ELECTRODES, P2 ELECTRODES, P3 ELECTRODES, U1 ADS1299, U10 ESP32-C3-WROOM-02, U2 ADS1299, U3 ADS1299, U9 LM3480-3.3

Commit message: Add fabrication outputs and update KiCad schematic, PCB, and ERC.
Co-authored-by: Cursor <cursoragent@cursor.com>
Parts:
- removed C1, C14, C15, C16, C2, C3, C33, C34, C35, C36, C37, C38, C39, C4, C40, C41, C42, C43, C53, C54, C55, C56, C57, C58, C59, C60: 4n7, Capacitor_SMD:C_0603_1608Metric, symbol Device:C
- removed C22, C69, C72: 0.1uF, Capacitor_SMD:C_0603_1608Metric, symbol EEG_BLE-rescue:C
- removed C23, C70, C73: 10uF, Capacitor_SMD:C_0603_1608Metric, symbol EEG_BLE-rescue:C
- removed R29, R30, R31, R32, R33, R34, R35, R36, R37, R38, R39, R40, R41, R42, R43, R44, R45, R46, R47, R48, R49, R9: 5k6, Resistor_SMD:R_0603_1608Metric, symbol Device:R
- added C20, C40, C60: 0.1uF, Capacitor_SMD:C_0402_1005Metric, symbol EEG_BLE-rescue:C
- added C21, C41, C61: 10uF, Capacitor_SMD:C_0603_1608Metric, symbol EEG_BLE-rescue:C
- added C24, C25, C26, C27, C28: 4n7, Capacitor_SMD:C_0402_1005Metric, symbol Device:C
- added R17: 5k6, Resistor_SMD:R_0603_1608Metric, symbol Device:R
- added R_GND2: 0R, Resistor_SMD:R_0603_1608Metric, symbol Device:R
- C1: renamed from C24; footprint Capacitor_SMD:C_0603_1608Metric -> Capacitor_SMD:C_0402_1005Metric
- C10, C11, C12, C29, C30, C31, C32, C44, C45, C46, C47, C48, C49, C5, C50, C51, C52, C6, C7, C8, C9: footprint Capacitor_SMD:C_0603_1608Metric -> Capacitor_SMD:C_0402_1005Metric
- C13: renamed from C17; footprint Capacitor_SMD:C_0603_1608Metric -> Capacitor_SMD:C_0402_1005Metric
- C14: renamed from C18; footprint Capacitor_SMD:C_0603_1608Metric -> Capacitor_SMD:C_0402_1005Metric
- C15: renamed from C20; footprint Capacitor_SMD:C_0603_1608Metric -> Capacitor_SMD:C_0402_1005Metric
- C16: renamed from C21; footprint Capacitor_SMD:C_0603_1608Metric -> Capacitor_SMD:C_0402_1005Metric
- C17: renamed from C25; footprint Capacitor_SMD:C_0603_1608Metric -> Capacitor_SMD:C_0402_1005Metric
- C18: renamed from C27; footprint Capacitor_SMD:C_0603_1608Metric -> Capacitor_SMD:C_0805_2012Metric
- C19: renamed from C28; footprint Capacitor_SMD:C_0603_1608Metric -> Capacitor_SMD:C_0402_1005Metric
- C2: renamed from C26; footprint Capacitor_SMD:C_0603_1608Metric -> Capacitor_SMD:C_0402_1005Metric
- C22: renamed from C71; footprint Capacitor_SMD:C_0603_1608Metric -> Capacitor_SMD:C_0402_1005Metric
- C23: renamed from C75; footprint Capacitor_SMD:C_0603_1608Metric -> Capacitor_SMD:C_0402_1005Metric
- C3: renamed from C19; footprint Capacitor_SMD:C_0603_1608Metric -> Capacitor_SMD:C_0402_1005Metric
- C33: renamed from C61; footprint Capacitor_SMD:C_0603_1608Metric -> Capacitor_SMD:C_0402_1005Metric
- C34: renamed from C62; footprint Capacitor_SMD:C_0603_1608Metric -> Capacitor_SMD:C_0402_1005Metric
- C35: renamed from C64; footprint Capacitor_SMD:C_0603_1608Metric -> Capacitor_SMD:C_0402_1005Metric
- C36: renamed from C66; footprint Capacitor_SMD:C_0603_1608Metric -> Capacitor_SMD:C_0402_1005Metric
- C37: renamed from C74; footprint Capacitor_SMD:C_0603_1608Metric -> Capacitor_SMD:C_0402_1005Metric
- C38: renamed from C77; footprint Capacitor_SMD:C_0603_1608Metric -> Capacitor_SMD:C_0805_2012Metric
- C39: renamed from C79; footprint Capacitor_SMD:C_0603_1608Metric -> Capacitor_SMD:C_0402_1005Metric
- C4: renamed from C13; footprint Capacitor_SMD:C_0603_1608Metric -> Capacitor_SMD:C_0402_1005Metric
- C42: renamed from C76; footprint Capacitor_SMD:C_0603_1608Metric -> Capacitor_SMD:C_0402_1005Metric
- C43: renamed from C80; footprint Capacitor_SMD:C_0603_1608Metric -> Capacitor_SMD:C_0402_1005Metric
- C53: renamed from C63; footprint Capacitor_SMD:C_0603_1608Metric -> Capacitor_SMD:C_0402_1005Metric
- C54: renamed from C65; footprint Capacitor_SMD:C_0603_1608Metric -> Capacitor_SMD:C_0402_1005Metric
- C55: renamed from C67; footprint Capacitor_SMD:C_0603_1608Metric -> Capacitor_SMD:C_0402_1005Metric
- C56: renamed from C68; footprint Capacitor_SMD:C_0603_1608Metric -> Capacitor_SMD:C_0402_1005Metric
- C57: renamed from C78; footprint Capacitor_SMD:C_0603_1608Metric -> Capacitor_SMD:C_0402_1005Metric
- C58: renamed from C81; footprint Capacitor_SMD:C_0603_1608Metric -> Capacitor_SMD:C_0805_2012Metric
- C59: renamed from C82; footprint Capacitor_SMD:C_0603_1608Metric -> Capacitor_SMD:C_0402_1005Metric
- C62: renamed from C218; footprint Capacitor_SMD:C_0603_1608Metric -> Capacitor_SMD:C_0402_1005Metric
- C63: renamed from C219; footprint Capacitor_SMD:C_0603_1608Metric -> Capacitor_SMD:C_0402_1005Metric
- C64: renamed from C220; value 1uF -> 10uF; footprint Capacitor_SMD:C_0603_1608Metric -> Capacitor_SMD:C_0402_1005Metric
- C65: renamed from C221; value 0.1uF -> 1uF; footprint Capacitor_SMD:C_0603_1608Metric -> Capacitor_SMD:C_0402_1005Metric
- U5: renamed from U9; footprint Package_TO_SOT_SMD:SOT-23 -> Package_TO_SOT_SMD:SOT-223-3_TabPin2
- renumbered R17 to R1, R1 to R2, R2 to R3, R3 to R4, R4 to R5, R5 to R6, R6 to R7, R7 to R8, R8 to R9, U10 to U4
Connections:
- net AGND: now also C32.1, C45.1, C46.1, C47.1, C49.2, C5.1, C50.2, C52.1, C6.1, C8.1, C9.2, C24.1, C25.1, C26.1, C27.1, C28.1, R_GND2.1; no longer C13.2, C14.2, C15.2, C16.2, C32.2, C33.2, C34.2, C35.2, C36.2, C45.2, C46.2, C47.2, C49.1, C5.2, C50.1, C52.2, C53.2, C54.2, C55.2, C56.2, C6.2, C8.2, C9.1, U1.20 (AVSS), U1.23 (AVSS), U1.24 (VREFP), U2.20 (AVSS), U2.23 (AVSS), U2.24 (VREFP), U3.20 (AVSS), U3.23 (AVSS), U3.24 (VREFP)
- net AVSS: now also C13.2, C14.2, C15.2, C16.2, C17.2, C18.2, C19.2, C33.2, C34.2, C35.2, C36.2, C37.2, C38.2, C39.2, C53.2, C54.2, C55.2, C56.2, C57.2, C58.2, C59.2, U1.20 (AVSS), U1.23 (AVSS), U1.25 (VREFN), U1.32 (AVSS), U2.20 (AVSS), U2.23 (AVSS), U2.25 (VREFN), U2.32 (AVSS), U3.20 (AVSS), U3.23 (AVSS), U3.25 (VREFN), U3.32 (AVSS), C20.1, C21.1, C40.1, C41.1, C60.1, C61.1, R_GND2.2
- net SRB_REF: now also C32.2, C52.2, R19.2, R28.2; no longer C10.1, C11.1, C44.2, C46.1, C47.1, C48.2, C49.2, C51.1, C52.1, C7.2, C9.2, R11.2, R12.2, R13.2, R14.2, R15.2, R16.2, U1.17 (SRB1), U2.17 (SRB1), U3.17 (SRB1)
- net at U1.1 (IN8N): no longer R13.1
- net at U1.11 (IN3N): no longer R14.1
- net at U1.13 (IN2N): no longer R12.1
- net at U1.15 (IN1N): no longer R11.1
- net at R9.1: now also C11.1, U1.16 (IN1P); no longer U1.2 (IN8P)
- net at U1.3 (IN7N): no longer R15.1
- net at R8.1: now also C10.1, U1.14 (IN2P); no longer U1.4 (IN7P)
- net at R10.1: now also U1.17 (SRB1); no longer U1.5 (IN6N)
- net at R7.1: now also C9.1, U1.12 (IN3P); no longer U1.6 (IN6P)
- net at R6.1: now also C8.2, U1.10 (IN4P); no longer U1.8 (IN5P)
- net at U1.9 (IN4N): no longer R16.1
- net at U3.8 (IN5P): now also C47.2, R23.1
- net at U3.2 (IN8P): now also C44.2, R20.1; no longer C31.1
- net at R27.2: now also P3.10 (P10); no longer P3.4 (P4)
- net at U3.10 (IN4P): now also C48.2, R24.1
- net at R28.1: now also U3.17 (SRB1); no longer U3.12 (IN3P)
- net at U3.16 (IN1P): now also C51.1, R27.1; no longer R26.1
- net at U3.4 (IN7P): now also C45.2, R21.1
- net at U3.6 (IN6P): now also C46.2, R22.1; no longer C32.1
- net at R25.2: now also P3.8 (P8); no longer P2.10 (P10)
- net at U2.10 (IN4P): now also R15.1, C28.2; no longer R21.1
- net at U2.14 (IN2P): now also C30.1, R17.1; no longer R19.1
- net at R18.1, U2.16 (IN1P): now also C31.1
- net at U2.4 (IN7P): now also R12.1, C25.2; no longer R24.1
- net at U2.8 (IN5P): now also R14.1, C27.2; no longer R22.1
- net at P3.7 (P7): now also R24.2
- net at P3.3 (P3): now also R20.2; no longer R26.2
- net at P3.5 (P5): now also R22.2; no longer R28.2
- net at P3.6 (P6): now also R23.2
- net at P3.9 (P9): now also R26.2
- net at P2.4 (P4): now also R12.2; no longer R19.2
- net at P2.9 (P9): now also R17.2; no longer R24.2
- net at P2.3 (P3): now also R11.2; no longer R18.2
- net at P2.5 (P5): now also R13.2; no longer R20.2
- net at R21.2: now also P3.4 (P4); no longer P2.6 (P6)
- net at P2.7 (P7): now also R15.2; no longer R22.2
- net at P2.8 (P8): now also R16.2; no longer R23.2
- new net: C4.2, R2.1, U1.2 (IN8P)
- new net: C20.2, C21.2, U1.24 (VREFP)
- new net: C5.2, R3.1, U1.4 (IN7P)
- new net: C6.2, R4.1, U1.6 (IN6P)
- new net: C7.2, R5.1, U1.8 (IN5P)
- new net: C24.2, R11.1, U2.2 (IN8P)
- new net: C50.1, R26.1, U3.14 (IN2P)
- new net: C49.1, R25.1, U3.12 (IN3P)
- new net: C60.2, C61.2, U3.24 (VREFP)
- new net: P2.10 (P10), R18.2
- new net: C26.2, R13.1, U2.6 (IN6P)
- new net: C29.1, R16.1, U2.12 (IN3P)
- new net: R19.1, U2.17 (SRB1)
- new net: C40.2, C41.2, U2.24 (VREFP)
- new net: P2.6 (P6), R14.2
- no-connect marks 33 -> 54
Other:
- note removed: "Do SRB1 and SRB2 need to be connected to something, f.ex: AGND?"
- moved on the sheet: C1, C13, C14, C15, C16, C17, C18, C19, C2, C22, C23, C3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
